File: DAC_ISINK_PMOD_Board_V1/DAC_ISINK_PMOD_Board_V1.kicad_sch (KiCad schematic)
At the start: 9 parts, among them P1 PMOD-Device-x2-Type-Generic-A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

Commit message: Manufacturing Data Generated.
Parts:
- added J3: Conn_01x04, Connector_Phoenix_MC:PhoenixContact_MC_1,5_4-G-3.5_1x04_P3.50mm_Horizontal, symbol Connector_Generic:Conn_01x04
- added R15: 100R, Resistor_SMD:R_0603_1608Metric, symbol Device:R
- C26, C27, C28: footprint Capacitor_SMD:C_0402_1005Metric -> Capacitor_SMD:C_0603_1608Metric
- R13, R7, R8: footprint Resistor_SMD:R_0402_1005Metric -> Resistor_SMD:R_0603_1608Metric
- R9: footprint (none) -> Resistor_SMD:R_0603_1608Metric
Connections:
- net 3V3_PMOD: now also R15.1
- net GND: now also J3.2 (Pin_2)
- net I_SINK: now also J3.3 (Pin_3)
- net LDAC_N: now also P1.4 (P4); no longer P1.3 (P3)
- net RESET_N: now also P1.3 (P3); no longer P1.4 (P4)
- net SCL: now also P1.2 (P2); no longer P1.1 (P1)
- net SDA: now also P1.1 (P1); no longer P1.2 (P2)
- net V_OUT_0: now also J3.1 (Pin_1)
- new net: J3.4 (Pin_4), R15.2
- no-connect marks 0 -> 4
